File: layout/kicad/simkarte.kicad_sch (KiCad schematic)
At the start: 12 parts, among them J1 SIM_Card, U1 ATtiny85-20PU, U2 ATtiny85-20PU

Commit message: C-Netz: Updated sim card layout to support memory card emulation.
A jumper must be switched in order to emulate the reset input.

Also added new service codes to the silk mask.
Parts:
- added JP1: Jumper_3_Bridged12, Jumper:SolderJumper-3_P1.3mm_Bridged12_RoundedPad1.0x1.5mm_NumberLabels, symbol Jumper:Jumper_3_Bridged12
Connections:
- net at TP7.1, U1.1 (~{RESET}/PB5), U2.1 (~{RESET}/PB5): now also JP1.1 (A); no longer J1.2 (RST)
- net at U2.7 (PB2): now also TP5.1, U1.7 (PB2), JP1.3 (B)
- new net: J1.2 (RST), JP1.2 (C)
Changed lines of the file:
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@@
   (junction (at 177.8 86.36) (diameter 0) (color 0 0 0 0)
   )
+  (junction (at 189.23 83.82) (diameter 0) (color 0 0 0 0)
+  )
+  (junction (at 173.99 81.28) (diameter 0) (color 0 0 0 0)
+  )
+  (junction (at 186.69 81.28) (diameter 0) (color 0 0 0 0)
+  )
+  (junction (at 170.18 78.74) (diameter 0) (color 0 0 0 0)
+  )
   (junction (at 191.77 86.36) (diameter 0) (color 0 0 0 0)
-  )
-  (junction (at 189.23 83.82) (diameter 0) (color 0 0 0 0)
-  )
-  (junction (at 173.99 81.28) (diameter 0) (color 0 0 0 0)
-  )
-  (junction (at 186.69 81.28) (diameter 0) (color 0 0 0 0)
   )
   (no_connect (at 203.2 83.82))
@@
     (stroke (width 0) (type default) (color 0 0 0 0))
   )
-  (wire (pts (xy 191.77 76.2) (xy 203.2 76.2))
-    (stroke (width 0) (type default) (color 0 0 0 0))
-  )
   (wire (pts (xy 186.69 78.74) (xy 186.69 81.28))
     (stroke (width 0) (type default) (color 0 0 0 0))
@@
     (stroke (width 0) (type default) (color 0 0 0 0))
   )
+  (wire (pts (xy 195.58 76.2) (xy 195.58 68.58))
+    (stroke (width 0) (type default) (color 0 0 0 0))
+  )
   (wire (pts (xy 195.58 86.36) (xy 203.2 86.36))
     (stroke (width 0) (type default) (color 0 0 0 0))
@@
     (stroke (width 0) (type default) (color 0 0 0 0))
   )
-  (wire (pts (xy 191.77 86.36) (xy 191.77 76.2))
+  (wire (pts (xy 185.42 62.23) (xy 191.77 62.23))
+    (stroke (width 0) (type default) (color 0 0 0 0))
+  )
+  (wire (pts (xy 203.2 76.2) (xy 195.58 76.2))
     (stroke (width 0) (type default) (color 0 0 0 0))
   )
@@
     (stroke (width 0) (type default) (color 0 0 0 0))
   )
+  (wire (pts (xy 170.18 78.74) (xy 170.18 125.73))
+    (stroke (width 0) (type default) (color 0 0 0 0))
+  )
   (wire (pts (xy 189.23 83.82) (xy 195.58 83.82))
     (stroke (width 0) (type default) (color 0 0 0 0))
@@
     (stroke (width 0) (type default) (color 0 0 0 0))
   )
+  (wire (pts (xy 191.77 74.93) (xy 191.77 86.36))
+    (stroke (width 0) (type default) (color 0 0 0 0))
+  )
   (wire (pts (xy 160.02 86.36) (xy 177.8 86.36))
     (stroke (width 0) (type default) (color 0 0 0 0))
@@
   )
   (wire (pts (xy 170.18 78.74) (xy 170.18 64.77))
+    (stroke (width 0) (type default) (color 0 0 0 0))
+  )
+  (wire (pts (xy 185.42 62.23) (xy 185.42 78.74))
+    (stroke (width 0) (type default) (color 0 0 0 0))
+  )
+  (wire (pts (xy 170.18 78.74) (xy 185.42 78.74))
+    (stroke (width 0) (type default) (color 0 0 0 0))
+  )
+  (wire (pts (xy 170.18 125.73) (xy 160.02 125.73))
     (stroke (width 0) (type default) (color 0 0 0 0))
   )
@@
     (pin "1")
   )
+  (symbol (lib_id "Jumper:Jumper_3_Bridged12") (at 191.77 68.58 90) (unit 1)
+    (in_bom yes) (on_board yes) (fields_autoplaced)
+    (property "Reference" "JP1" (id 0) (at 189.23 67.3099 90)
+      (effects (font (size 1.27 1.27)) (justify left))
+    )
+    (property "Value" "Jumper_3_Bridged12" (id 1) (at 189.23 69.8499 90)
+      (effects (font (size 1.27 1.27)) (justify left))
+    )
+    (property "Footprint" "Jumper:SolderJumper-3_P1.3mm_Bridged12_RoundedPad1.0x1.5mm_NumberLabels" (id 2) (at 191.77 68.58 0)
+      (effects (font (size 1.27 1.27)) hide)
+    )
+    (property "Datasheet" "~" (id 3) (at 191.77 68.58 0)
+      (effects (font (size 1.27 1.27)) hide)
+    )
+    (pin "1")
+    (pin "2")
+    (pin "3")
+  )
   (sheet_instances
     (path "/" (page "1"))
@@
       (reference "J1") (unit 1) (value "SIM_Card") (footprint "simkarte:SIM-Pads")
     )
+    (path "/fbeca373-4216-4e9d-b531-72235a36bc1e"
+      (reference "JP1") (unit 1) (value "Jumper_3_Bridged12") (footprint "Jumper:SolderJumper-3_P1.3mm_Bridged12_RoundedPad1.0x1.5mm_NumberLabels")
+    )
     (path "/00000000-0000-0000-0000-0000629b0678"
